File: hw/teacup-t41.kicad_pcb (KiCad board)
At the start: 4 copper layers, 86.2 x 56.2 mm, 123 parts, among them IC1 T41NQ, J1 USB Type-C, J10 AudioJack4_Ground, J11 Conn_01x04_Pin, J12 Conn_01x04_Pin, J13 SFW15R-2STE1LF, J14 Conn_01x02_MountingPin, J15 Conn_01x03_MountingPin, J16 Conn_01x03_MountingPin, J2 Micro_SD_Card, J3 USB_A, J4 Conn_02x08_Odd_Even, J5 UART, J6 Conn_02x07_Odd_Even, J7 Conn_02x07_Odd_Even, J8 DC_IN, J9 Conn_01x02_MountingPin, SW2 SW_SPDT, U1 AZ1117-3.3, U2 AZ1117-1.8, U4 W25Q32JVSS, U5 W25Q32JVSS, U6 SY8089A1AAC, U7 SY8089A1AAC, Y1 24 MHz

Commit message: Route PCB (FreeRouting ~83%) + draft manufacturing outputs
pcbnew placement of 20 new parts on B.Cu, Specctra DSN export,
FreeRouting v1.9.0 autoroute under xvfb (13:45 route + opt, ~50%
improvement), SES import: 940 traces + 120 vias. Zones refilled.

NOT fab-ready: 78 nets unrouted, 7 courtyard overlaps (blind bottom
placement), 3 shorts, MIPI not impedance-controlled. DRC report in
hw/Manufacturing/. BOM + position complete and correct. Needs GUI
finishing before fab. scripts/gen_pcb_import_route.py + gen_manufacturing.sh.
Parts:
- C47, C48, C49, C50, C51, C52, C53, C54, C55, L1, L2, R26, R27, R28, R29, R30, R31, R32, U6, U7: moved to B.Cu
- moved R30 36.4 mm to (176.0, 101.0), turned to 180 degrees
- moved R32 31.8 mm to (192.0, 101.0), turned to 180 degrees
- moved C48 30.8 mm to (180.0, 98.0), turned to 180 degrees
- moved R29 29.7 mm to (180.0, 101.0), turned to 180 degrees
- moved C51 29.7 mm to (192.0, 98.0), turned to 180 degrees
- moved C52 28.7 mm to (196.0, 98.0), turned to 180 degrees
- moved U7 28.3 mm to (200.0, 98.0), turned to 180 degrees
- moved C49 27.8 mm to (184.0, 101.0), turned to 180 degrees
- moved C55 27.7 mm to (208.0, 98.0), turned to 180 degrees
- moved L2 27.6 mm to (204.0, 98.0), turned to 180 degrees
- moved U6 27.6 mm to (184.0, 98.0), turned to 180 degrees
- moved C50 27.2 mm to (188.0, 101.0), turned to 180 degrees
- moved L1 26.9 mm to (188.0, 98.0), turned to 180 degrees
- moved R31 26.1 mm to (196.0, 101.0), turned to 180 degrees
- moved C53 25.6 mm to (200.0, 101.0), turned to 180 degrees
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Routing:
- net +3V3: track 0.00 -> 232.8 mm, vias 0 -> 26
- net +5V: track 0.00 -> 162.1 mm, vias 0 -> 2
- net /MICLP: track 0.00 -> 104.6 mm, vias 0 -> 1
- net GND: track 0.00 -> 104.1 mm, vias 0 -> 45
- net /NOR_CK: track 0.00 -> 72.4 mm, vias 0 -> 1
- net /MMC0_D1: track 0.00 -> 65.9 mm, vias 0 -> 2
- net /NOR_HOLD: track 0.00 -> 65.3 mm, vias 0 -> 2
- net /MMC0_CMD: track 0.00 -> 58.5 mm, vias 0 -> 2
- net /MMC0_D2: track 0.00 -> 57.2 mm
- net /UART0_RXD: track 0.00 -> 55.5 mm, vias 0 -> 2
- net /MDIO: track 0.00 -> 54.4 mm, vias 0 -> 2
- net /UART0_TXD: track 0.00 -> 52.2 mm, vias 0 -> 1
- net +1V35: track 0.00 -> 50.9 mm, vias 0 -> 2
- net /MDCK: track 0.00 -> 47.4 mm, vias 0 -> 1
- net +0V8: track 0.00 -> 46.7 mm, vias 0 -> 6
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