File: hw/teacup-carrier.kicad_sch (KiCad schematic)
At the start: 91 parts, among them J1 AH58893-T9B10-3F, J2 TYPE-C-31-M-12, J20 HDR_J20, J21 HDR_J21, J22 HDR_J22, J23 HDR_J23, J24 HDR_J24, J25 HDR_J25, J26 HDR_J26, J27 HDR_J27, J28 HDR_J28, J29 HDR_J29, J3 TE_292303-7, J30 HDR_J30, J4 Hirose_DM3D-SF, J5 Wuerth_694106301002, J6 AudioJack4_Ground, J7 SFW15R-2STE1LF, J8 SFW15R-2STE1LF, J9 TYPE-C-31-M-12, Q1 AO3401A, Q2 AO3401A, SW1 SSSS711403, SW2 SSSS711403, U1 AP62600SJ-7, U10 TS5A3166, U11 DIP-8 Socket, U12 TPS2053BDR, U13 W25Q32JVSS, U14 TPS22990DMLR, U15 TCA9555PWR, U2 AP62300WU-7, U3 MCP4661-104E_ST, U4 TPS22990DMLR, U5 AZ1117CH-3.3TRG1, U6 AZ1117CH-1.8TRG1, U7 AP62300WU-7, U8 ESP32-S3-WROOM-1-N16R2, U9 TS5A3166

Commit message: Carrier board: break out all remaining J1 pins to spare headers
Per explicit direction: every J1 pin still unused after the SS8
superset breakout (unit 4's 170-192 tail + units 5-6, 119 pins total)
now gets a raw SPARE_P<n> global label (n = the literal connector pin
number) routed to 5 new headers (J31-J35, grouped by connector unit
for traceability). No function is assumed for these -- reserved for
whatever a future interposer or bring-up need wants. Each header's
GND reference pin ties to the common GND net rather than consuming a
J1 position, so it's free against the pin/ground budget; this does
trade away some of SS8's "ground is fill" signal-integrity margin on
this connector for maximum future flexibility, which is the point.

Verified: 0 overlaps, netlist diff shows only the 119 new J1 net
assignments + 5 new header refs added (nothing else moved), ERC total
violation count unchanged (426 before/after -- the pin_not_connected
violations these pins carried became the board's existing pin_to_pin
"unspecified pin type" warning class instead, no new categories).
Parts:
- added J31: HDR_J31, Connector_PinHeader_2.54mm:PinHeader_1x24_P2.54mm_Vertical, symbol Connector_Generic:Conn_01x24
- added J32: HDR_J32, Connector_PinHeader_2.54mm:PinHeader_1x25_P2.54mm_Vertical, symbol Connector_Generic:Conn_01x25
- added J33: HDR_J33, Connector_PinHeader_2.54mm:PinHeader_1x25_P2.54mm_Vertical, symbol Connector_Generic:Conn_01x25
- added J34: HDR_J34, Connector_PinHeader_2.54mm:PinHeader_1x25_P2.54mm_Vertical, symbol Connector_Generic:Conn_01x25
- added J35: HDR_J35, Connector_PinHeader_2.54mm:PinHeader_1x25_P2.54mm_Vertical, symbol Connector_Generic:Conn_01x25
Connections:
- net GND: now also J31.1 (Pin_1), J32.1 (Pin_1), J33.1 (Pin_1), J34.1 (Pin_1), J35.1 (Pin_1)
- net SPARE_P193: now reaches J1.193 (P193)
- net SPARE_P193: now also J32.2 (Pin_2)
- net SPARE_P194: now reaches J1.194 (P194)
- net SPARE_P194: now also J32.3 (Pin_3)
- net SPARE_P195: now reaches J1.195 (P195)
- net SPARE_P195: now also J32.4 (Pin_4)
- net SPARE_P196: now reaches J1.196 (P196)
- net SPARE_P196: now also J32.5 (Pin_5)
- net SPARE_P197: now reaches J1.197 (P197)
- net SPARE_P197: now also J32.6 (Pin_6)
- net SPARE_P198: now reaches J1.198 (P198)
- net SPARE_P198: now also J32.7 (Pin_7)
- net SPARE_P199: now reaches J1.199 (P199)
- net SPARE_P199: now also J32.8 (Pin_8)
- net SPARE_P200: now reaches J1.200 (P200)
- net SPARE_P200: now also J32.9 (Pin_9)
- net SPARE_P201: now reaches J1.201 (P201)
- net SPARE_P201: now also J32.10 (Pin_10)
- net SPARE_P202: now reaches J1.202 (P202)
- net SPARE_P202: now also J32.11 (Pin_11)
- net SPARE_P203: now reaches J1.203 (P203)
- net SPARE_P203: now also J32.12 (Pin_12)
- net SPARE_P204: now reaches J1.204 (P204)
- net SPARE_P204: now also J32.13 (Pin_13)
- net SPARE_P205: now reaches J1.205 (P205)
- net SPARE_P205: now also J32.14 (Pin_14)
- net SPARE_P206: now reaches J1.206 (P206)
- net SPARE_P206: now also J32.15 (Pin_15)
- net SPARE_P207: now reaches J1.207 (P207)
- net SPARE_P207: now also J32.16 (Pin_16)
- net SPARE_P208: now reaches J1.208 (P208)
- net SPARE_P208: now also J32.17 (Pin_17)
- net SPARE_P209: now reaches J1.209 (P209)
- net SPARE_P209: now also J32.18 (Pin_18)
- net SPARE_P210: now reaches J1.210 (P210)
- net SPARE_P210: now also J32.19 (Pin_19)
- net SPARE_P211: now reaches J1.211 (P211)
- net SPARE_P211: now also J32.20 (Pin_20)
- net SPARE_P212: now reaches J1.212 (P212)
- net SPARE_P212: now also J32.21 (Pin_21)
- net SPARE_P213: now reaches J1.213 (P213)
- net SPARE_P213: now also J32.22 (Pin_22)
- net SPARE_P214: now reaches J1.214 (P214)
- net SPARE_P214: now also J32.23 (Pin_23)
- net SPARE_P215: now reaches J1.215 (P215)
- net SPARE_P215: now also J32.24 (Pin_24)
- net SPARE_P216: now reaches J1.216 (P216)
- net SPARE_P216: now also J32.25 (Pin_25)
- net SPARE_P217: now reaches J1.217 (P217)
- net SPARE_P217: now also J33.2 (Pin_2)
- net SPARE_P218: now reaches J1.218 (P218)
- net SPARE_P218: now also J33.3 (Pin_3)
- net SPARE_P219: now reaches J1.219 (P219)
- net SPARE_P219: now also J33.4 (Pin_4)
- net SPARE_P220: now reaches J1.220 (P220)
- net SPARE_P220: now also J33.5 (Pin_5)
- net SPARE_P221: now reaches J1.221 (P221)
- net SPARE_P221: now also J33.6 (Pin_6)
- net SPARE_P222: now reaches J1.222 (P222)
- net SPARE_P222: now also J33.7 (Pin_7)
- net SPARE_P223: now reaches J1.223 (P223)
- net SPARE_P223: now also J33.8 (Pin_8)
- net SPARE_P224: now reaches J1.224 (P224)
- net SPARE_P224: now also J33.9 (Pin_9)
- net SPARE_P225: now reaches J1.225 (P225)
- net SPARE_P225: now also J33.10 (Pin_10)
- net SPARE_P226: now reaches J1.226 (P226)
- net SPARE_P226: now also J33.11 (Pin_11)
- net SPARE_P227: now reaches J1.227 (P227)
- net SPARE_P227: now also J33.12 (Pin_12)
- net SPARE_P228: now reaches J1.228 (P228)
- net SPARE_P228: now also J33.13 (Pin_13)
- net SPARE_P229: now reaches J1.229 (P229)
- net SPARE_P229: now also J33.14 (Pin_14)
- net SPARE_P230: now reaches J1.230 (P230)
- net SPARE_P230: now also J33.15 (Pin_15)
- net SPARE_P231: now reaches J1.231 (P231)
- net SPARE_P231: now also J33.16 (Pin_16)
- net SPARE_P232: now reaches J1.232 (P232)
- net SPARE_P232: now also J33.17 (Pin_17)
- net SPARE_P233: now reaches J1.233 (P233)
- net SPARE_P233: now also J33.18 (Pin_18)
- net SPARE_P234: now reaches J1.234 (P234)
- net SPARE_P234: now also J33.19 (Pin_19)
- net SPARE_P235: now reaches J1.235 (P235)
- net SPARE_P235: now also J33.20 (Pin_20)
- net SPARE_P236: now reaches J1.236 (P236)
- net SPARE_P236: now also J33.21 (Pin_21)
- net SPARE_P237: now reaches J1.237 (P237)
- net SPARE_P237: now also J33.22 (Pin_22)
- net SPARE_P238: now reaches J1.238 (P238)
- net SPARE_P238: now also J33.23 (Pin_23)
- net SPARE_P239: now reaches J1.239 (P239)
- net SPARE_P239: now also J33.24 (Pin_24)
- net SPARE_P240: now reaches J1.240 (P240)
- net SPARE_P240: now also J33.25 (Pin_25)
- net SPARE_P241: now reaches J1.241 (P241)
- net SPARE_P241: now also J34.2 (Pin_2)
- net SPARE_P242: now reaches J1.242 (P242)
- net SPARE_P242: now also J34.3 (Pin_3)
- net SPARE_P243: now reaches J1.243 (P243)
- net SPARE_P243: now also J34.4 (Pin_4)
- net SPARE_P244: now reaches J1.244 (P244)
- net SPARE_P244: now also J34.5 (Pin_5)
- net SPARE_P245: now reaches J1.245 (P245)
- net SPARE_P245: now also J34.6 (Pin_6)
- net SPARE_P246: now reaches J1.246 (P246)
- net SPARE_P246: now also J34.7 (Pin_7)
- net SPARE_P247: now reaches J1.247 (P247)
- net SPARE_P247: now also J34.8 (Pin_8)
- net SPARE_P248: now reaches J1.248 (P248)
- net SPARE_P248: now also J34.9 (Pin_9)
- net SPARE_P249: now reaches J1.249 (P249)
- net SPARE_P249: now also J34.10 (Pin_10)
- net SPARE_P250: now reaches J1.250 (P250)
- net SPARE_P250: now also J34.11 (Pin_11)
- net SPARE_P251: now reaches J1.251 (P251)
- net SPARE_P251: now also J34.12 (Pin_12)
- net SPARE_P252: now reaches J1.252 (P252)
- net SPARE_P252: now also J34.13 (Pin_13)
- net SPARE_P253: now reaches J1.253 (P253)
- net SPARE_P253: now also J34.14 (Pin_14)
- net SPARE_P254: now reaches J1.254 (P254)
- net SPARE_P254: now also J34.15 (Pin_15)
- net SPARE_P255: now reaches J1.255 (P255)
- net SPARE_P255: now also J34.16 (Pin_16)
- net SPARE_P256: now reaches J1.256 (P256)
- net SPARE_P256: now also J34.17 (Pin_17)
- net SPARE_P257: now reaches J1.257 (P257)
- net SPARE_P257: now also J34.18 (Pin_18)
- net SPARE_P258: now reaches J1.258 (P258)
- net SPARE_P258: now also J34.19 (Pin_19)
- net SPARE_P259: now reaches J1.259 (P259)
- net SPARE_P259: now also J34.20 (Pin_20)
- net SPARE_P260: now reaches J1.260 (P260)
- net SPARE_P260: now also J34.21 (Pin_21)
- net SPARE_P261: now reaches J1.261 (P261)
- net SPARE_P261: now also J34.22 (Pin_22)
- net SPARE_P262: now reaches J1.262 (P262)
- net SPARE_P262: now also J34.23 (Pin_23)
- net SPARE_P263: now reaches J1.263 (P263)
- net SPARE_P263: now also J34.24 (Pin_24)
- net SPARE_P264: now reaches J1.264 (P264)
- net SPARE_P264: now also J34.25 (Pin_25)
- net SPARE_P265: now reaches J1.265 (P265)
- net SPARE_P265: now also J35.2 (Pin_2)
- net SPARE_P266: now reaches J1.266 (P266)
- net SPARE_P266: now also J35.3 (Pin_3)
- net SPARE_P267: now reaches J1.267 (P267)
- net SPARE_P267: now also J35.4 (Pin_4)
- net SPARE_P268: now reaches J1.268 (P268)
- net SPARE_P268: now also J35.5 (Pin_5)
- net SPARE_P269: now reaches J1.269 (P269)
- net SPARE_P269: now also J35.6 (Pin_6)
- net SPARE_P270: now reaches J1.270 (P270)
- net SPARE_P270: now also J35.7 (Pin_7)
- net SPARE_P271: now reaches J1.271 (P271)
- net SPARE_P271: now also J35.8 (Pin_8)
- net SPARE_P272: now reaches J1.272 (P272)
- net SPARE_P272: now also J35.9 (Pin_9)
- net SPARE_P273: now reaches J1.273 (P273)
- net SPARE_P273: now also J35.10 (Pin_10)
- net SPARE_P274: now reaches J1.274 (P274)
- net SPARE_P274: now also J35.11 (Pin_11)
- net SPARE_P275: now reaches J1.275 (P275)
- net SPARE_P275: now also J35.12 (Pin_12)
- net SPARE_P276: now reaches J1.276 (P276)
- net SPARE_P276: now also J35.13 (Pin_13)
- net SPARE_P277: now reaches J1.277 (P277)
- net SPARE_P277: now also J35.14 (Pin_14)
- net SPARE_P278: now reaches J1.278 (P278)
- net SPARE_P278: now also J35.15 (Pin_15)
- net SPARE_P279: now reaches J1.279 (P279)
- net SPARE_P279: now also J35.16 (Pin_16)
- net SPARE_P280: now reaches J1.280 (P280)
- net SPARE_P280: now also J35.17 (Pin_17)
- net SPARE_P281: now reaches J1.281 (P281)
- net SPARE_P281: now also J35.18 (Pin_18)
- net SPARE_P282: now reaches J1.282 (P282)
- net SPARE_P282: now also J35.19 (Pin_19)
- net SPARE_P283: now reaches J1.283 (P283)
- net SPARE_P283: now also J35.20 (Pin_20)
- net SPARE_P284: now reaches J1.284 (P284)
- net SPARE_P284: now also J35.21 (Pin_21)
- net SPARE_P285: now reaches J1.285 (P285)
- net SPARE_P285: now also J35.22 (Pin_22)
- net SPARE_P286: now reaches J1.286 (P286)
- net SPARE_P286: now also J35.23 (Pin_23)
- net SPARE_P287: now reaches J1.287 (P287)
- net SPARE_P287: now also J35.24 (Pin_24)
- net SPARE_P288: now reaches J1.288 (P288)
- net SPARE_P288: now also J35.25 (Pin_25)
- net SPARE_P170: now reaches J1.170 (P170)
- net SPARE_P170: now also J31.2 (Pin_2)
- net SPARE_P171: now reaches J1.171 (P171)
- net SPARE_P171: now also J31.3 (Pin_3)
- net SPARE_P172: now reaches J1.172 (P172)
- net SPARE_P172: now also J31.4 (Pin_4)
- net SPARE_P173: now reaches J1.173 (P173)
- net SPARE_P173: now also J31.5 (Pin_5)
- net SPARE_P174: now reaches J1.174 (P174)
- net SPARE_P174: now also J31.6 (Pin_6)
- net SPARE_P175: now reaches J1.175 (P175)
- net SPARE_P175: now also J31.7 (Pin_7)
- net SPARE_P176: now reaches J1.176 (P176)
- net SPARE_P176: now also J31.8 (Pin_8)
- net SPARE_P177: now reaches J1.177 (P177)
- net SPARE_P177: now also J31.9 (Pin_9)
- net SPARE_P178: now reaches J1.178 (P178)
- net SPARE_P178: now also J31.10 (Pin_10)
- net SPARE_P179: now reaches J1.179 (P179)
- net SPARE_P179: now also J31.11 (Pin_11)
- net SPARE_P180: now reaches J1.180 (P180)
- net SPARE_P180: now also J31.12 (Pin_12)
- net SPARE_P181: now reaches J1.181 (P181)
- net SPARE_P181: now also J31.13 (Pin_13)
- net SPARE_P182: now reaches J1.182 (P182)
- net SPARE_P182: now also J31.14 (Pin_14)
- net SPARE_P183: now reaches J1.183 (P183)
- net SPARE_P183: now also J31.15 (Pin_15)
- net SPARE_P184: now reaches J1.184 (P184)
- net SPARE_P184: now also J31.16 (Pin_16)
- net SPARE_P185: now reaches J1.185 (P185)
- net SPARE_P185: now also J31.17 (Pin_17)
- net SPARE_P186: now reaches J1.186 (P186)
- net SPARE_P186: now also J31.18 (Pin_18)
- net SPARE_P187: now reaches J1.187 (P187)
- net SPARE_P187: now also J31.19 (Pin_19)
- net SPARE_P188: now reaches J1.188 (P188)
- net SPARE_P188: now also J31.20 (Pin_20)
- net SPARE_P189: now reaches J1.189 (P189)
- net SPARE_P189: now also J31.21 (Pin_21)
- net SPARE_P190: now reaches J1.190 (P190)
- net SPARE_P190: now also J31.22 (Pin_22)
- net SPARE_P191: now reaches J1.191 (P191)
- net SPARE_P191: now also J31.23 (Pin_23)
- net SPARE_P192: now reaches J1.192 (P192)
- net SPARE_P192: now also J31.24 (Pin_24)
Other:
- note added: "J1 SPARE (P170-192)"
- note added: "J1 SPARE (P193-216)"
- note added: "J1 SPARE (P217-240)"
- note added: "J1 SPARE (P241-264)"
- note added: "J1 SPARE (P265-288)"
