File: hw/teacup-carrier.kicad_sch (KiCad schematic)
At the start: 128 parts, among them J1 AH58893-T9B10-3F, J2 TYPE-C-31-M-12, J20 HDR_J20, J21 HDR_J21, J22 HDR_J22, J23 HDR_J23, J24 HDR_J24, J25 HDR_J25, J26 HDR_J26, J27 HDR_J27, J28 HDR_J28, J29 HDR_J29, J3 TE_292303-7, J30 HDR_J30, J31 HDR_J31, J32 HDR_J32, J33 HDR_J33, J34 HDR_J34, J35 HDR_J35, J4 Hirose_DM3D-SF, J5 Wuerth_694106301002, J6 AudioJack4_Ground, J7 SFW15R-2STE1LF, J8 SFW15R-2STE1LF, J9 TYPE-C-31-M-12, Q1 AO3401A, Q2 AO3401A, SW1 SSSS711403, SW2 SSSS711403, U1 AP62600SJ-7, U10 TS5A3166, U11 DIP-8 Socket, U12 TPS2053BDR, U13 W25Q32JVSS, U14 TPS22990DMLR, U15 TCA9555PWR, U2 AP62300WU-7, U3 MCP4661-104E_ST, U4 TPS22990DMLR, U5 AZ1117CH-3.3TRG1, U6 AZ1117CH-1.8TRG1, U7 AP62300WU-7, U8 ESP32-S3-WROOM-1-N16R2, U9 TS5A3166

Commit message: Fix D1/D2 and U13 footprint references (didn't exist in any library)
Found while auditing every footprint reference in CONNECTIONS.txt against
the actual installed libraries (fp-lib-table + on-disk .kicad_mod files),
prompted by the earlier PCB pass's substituted-footprint workaround note:

- D1/D2 (PMEG2010ER): hardcoded Diode_SMD:D_SOD-123W, which doesn't exist
  anywhere, and Diode_SMD wasn't even registered in fp-lib-table. Fixed to
  Diode_SMD:Nexperia_CFP3_SOD-123W (the real footprint for this Nexperia
  part's actual package) and registered the library.
- U13 (W25Q32JVSS): hardcoded Package_SO:SOIC-8_5.23x5.23mm_P1.27mm --
  close but not the real footprint name, Package_SO:SOIC-8_5.3x5.3mm_P1.27mm.

Verified: netlist diff shows only these 3 footprint string changes,
nothing else moved (component count, all pin-net assignments unchanged).
ERC footprint_link_issues: 3 -> 0, no other category changed. PCB rebuild:
still just the 1 expected J6 case, DRC unchanged at 20 pre-existing
fine-pitch clearance violations. Schematic quadrant layout still at 0mm
drift.
Parts:
- D1, D2: footprint Diode_SMD:D_SOD-123W -> Diode_SMD:Nexperia_CFP3_SOD-123W
- U13: footprint Package_SO:SOIC-8_5.23x5.23mm_P1.27mm -> Package_SO:SOIC-8_5.3x5.3mm_P1.27mm
Changed lines of the file:
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@@
 		(property "Reference" "D1" (at 142.24 34.29 0) (effects (font (size 1.27 1.27))))
 		(property "Value" "PMEG2010ER" (at 142.24 41.91 0) (effects (font (size 1.27 1.27))))
-		(property "Footprint" "Diode_SMD:D_SOD-123W" (at 142.24 38.1 0) (effects (font (size 1.27 1.27)) hide))
+		(property "Footprint" "Diode_SMD:Nexperia_CFP3_SOD-123W" (at 142.24 38.1 0) (effects (font (size 1.27 1.27)) hide))
 	)
 	(symbol (lib_id "Device:D_Schottky") (at 142.24 53.34 0) (unit 1)
 		(property "Reference" "D2" (at 142.24 49.53 0) (effects (font (size 1.27 1.27))))
 		(property "Value" "PMEG2010ER" (at 142.24 57.15 0) (effects (font (size 1.27 1.27))))
-		(property "Footprint" "Diode_SMD:D_SOD-123W" (at 142.24 53.34 0) (effects (font (size 1.27 1.27)) hide))
+		(property "Footprint" "Diode_SMD:Nexperia_CFP3_SOD-123W" (at 142.24 53.34 0) (effects (font (size 1.27 1.27)) hide))
 	)
 	(symbol (lib_id "Regulator_Linear:L7805") (at 195.58 45.72 0) (unit 1)
@@
 		(property "Reference" "U13" (at 473.71 172.72 0) (effects (font (size 1.27 1.27))))
 		(property "Value" "W25Q32JVSS" (at 473.71 175.26 0) (effects (font (size 1.27 1.27))))
-		(property "Footprint" "Package_SO:SOIC-8_5.23x5.23mm_P1.27mm" (at 486.41 185.42 0) (effects (font (size 1.27 1.27)) hide))
+		(property "Footprint" "Package_SO:SOIC-8_5.3x5.3mm_P1.27mm" (at 486.41 185.42 0) (effects (font (size 1.27 1.27)) hide))
 	)
 	(symbol (lib_id "power:GND") (at 486.41 195.58 0) (unit 1)

Commit message: Confirm C13/C23 at 1nF, drop the _TBD marker
C13/C23 set the slew-rate/inrush-limiting CT capacitor on U4/U14
(TPS22990DMLR load switches, SS9). Verified 1nF against TI's own
TPS22990 datasheet, which uses this same 1000pF value as its reference
design default for this exact pin -- the placeholder wasn't wrong, just
unconfirmed against the datasheet until now.

Verified: netlist diff shows only these 2 value string changes, zero
pin-net changes. ERC unchanged at 429 violations. Schematic layout still
at 0mm drift.
Parts:
- C13, C23: value 1nF_TBD -> 1nF
Changed lines of the file:
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@@
 	(symbol (lib_id "Device:C") (at 172.72 147.32 0) (unit 1)
 		(property "Reference" "C13" (at 177.8 146.05 0) (effects (font (size 1.27 1.27))))
-		(property "Value" "1nF_TBD" (at 177.8 148.59 0) (effects (font (size 1.27 1.27))))
+		(property "Value" "1nF" (at 177.8 148.59 0) (effects (font (size 1.27 1.27))))
 		(property "Footprint" "Capacitor_SMD:C_0402_1005Metric" (at 172.72 147.32 0) (effects (font (size 1.27 1.27)) hide))
 	)
@@
 	(symbol (lib_id "Device:C") (at 248.92 147.32 0) (unit 1)
 		(property "Reference" "C23" (at 254 146.05 0) (effects (font (size 1.27 1.27))))
-		(property "Value" "1nF_TBD" (at 254 148.59 0) (effects (font (size 1.27 1.27))))
+		(property "Value" "1nF" (at 254 148.59 0) (effects (font (size 1.27 1.27))))
 		(property "Footprint" "Capacitor_SMD:C_0402_1005Metric" (at 248.92 147.32 0) (effects (font (size 1.27 1.27)) hide))
 	)
