File: hw/teacup-carrier.kicad_pcb (KiCad board)
At the start: 4 copper layers, 280 x 240 mm, 128 parts, among them J1 AH58893-T9B10-3F, J2 TYPE-C-31-M-12, J20 HDR_J20, J21 HDR_J21, J22 HDR_J22, J23 HDR_J23, J24 HDR_J24, J25 HDR_J25, J26 HDR_J26, J27 HDR_J27, J28 HDR_J28, J29 HDR_J29, J3 TE_292303-7, J30 HDR_J30, J31 HDR_J31, J32 HDR_J32, J33 HDR_J33, J34 HDR_J34, J35 HDR_J35, J4 Hirose_DM3D-SF, J5 Wuerth_694106301002, J6 AudioJack4_Ground, J7 SFW15R-2STE1LF, J8 SFW15R-2STE1LF, J9 TYPE-C-31-M-12, Q1 AO3401A, Q2 AO3401A, SW1 SSSS711403, SW2 SSSS711403, U1 AP62600SJ-7, U10 TS5A3166, U11 DIP-8 Socket, U12 TPS2053BDR, U13 W25Q32JVSS, U14 TPS22990DMLR, U15 TCA9555PWR, U2 AP62300WU-7, U3 MCP4661-104E_ST, U4 TPS22990DMLR, U5 AZ1117CH-3.3TRG1, U6 AZ1117CH-1.8TRG1, U7 AP62300WU-7, U8 ESP32-S3-WROOM-1-N16R2, U9 TS5A3166

Commit message: Carrier board: audio/FPC pinout fixes matching 3.3, SW2 remap, UART1 breakout, real PCB layout
Schematic fixes (verified pin-for-pin against TeaCup(C)3.3's real netlist,
not assumed):
- J6 audio jack: R1/R2 -> HPOUTL/GND, S -> MICLP, matching 3.3's J10 exactly
  (previous wiring incorrectly tied GND to a schematic pin, G, with no
  matching pad on the real Jack_3.5mm_PJ320D_Horizontal footprint).
- J7/J8 FPC camera connectors: full pin-for-pin remap to match 3.3's real
  J13 pinout -- the previous "standard RPi/Arducam" pinout had power/ground
  swapped, clock/data lanes in the wrong order, and reversed differential
  polarity throughout. Added JP11/JP12 sensor-enable select jumpers
  (GPIO vs hardwired +3V3), replicating 3.3's J15.
- J1 MIPI0/MIPI1 pin order on the connector reordered (CLK/D1/D0, P-before-N)
  to match J7/J8's now-fixed order, so routing between them doesn't need to
  cross over itself.
- HPOUTL relocated from J1 pin 58 (isolated, far from any other audio net)
  down to sit beside MICLP at pins 170-172, geography-first per
  UNIVERSAL.md SS8.
- SW2 (manual power-override switch) throw1/throw4 swapped: throw1 now
  forces ALT, throw4 now forces BMC.
- New J36 header breaks out UART1 (the BMC-ESP32<->J1 console link) for
  external monitoring, same as UART0/2/3 already had.

All verified via isolated before/after ERC diffs -- each change nets to
either 0 or a fully-explained delta against the 429-violation baseline,
never an unexplained regression.

PCB: teacup-carrier.kicad_pcb replaced with the manually-laid-out board
(previously developed as a separate merge-test attempt): real component
placement grouped by circuit block, board outline resized twice to
snugly enclose the layout, GND copper pour on both F.Cu and B.Cu, and
mounting holes repositioned to match. The old rough auto-placed board is
gone.
Parts:
- added H1: MountingHole_Pad, MountingHole_2.7mm_M2.5_Pad_Via, F.Cu at (21.2, 27.4)
- added H2: MountingHole_Pad, MountingHole_2.7mm_M2.5_Pad_Via, F.Cu at (271.9, 27.4)
- added H3: MountingHole_Pad, MountingHole_2.7mm_M2.5_Pad_Via, F.Cu at (21.2, 138.8)
- added H4: MountingHole_Pad, MountingHole_2.7mm_M2.5_Pad_Via, F.Cu at (271.9, 138.8)
- added J36: HDR_J36, PinHeader_1x03_P2.54mm_Vertical, F.Cu at (181.7, 138.1)
- added JP11: EN_SEL, PinHeader_1x03_P2.54mm_Vertical_SMD_Pin1Left, F.Cu at (241.0, 124.0)
- added JP12: EN_SEL, PinHeader_1x03_P2.54mm_Vertical_SMD_Pin1Left, F.Cu at (253.5, 124.0)
- J31: footprint PinHeader_2x12_P2.54mm_Vertical -> PinHeader_2x11_P2.54mm_Vertical
- moved J4 133.5 mm to (215.7, 131.8)
- moved J6 128.9 mm to (199.1, 133.6), turned to 90 degrees
- moved J8 128.4 mm to (257.9, 134.4)
- moved J7 128.4 mm to (235.7, 134.3)
- moved U5 121.9 mm to (36.6, 57.3)
- moved C17 121.6 mm to (46.6, 75.0), turned to 180 degrees
- moved R5 120.9 mm to (50.5, 76.5), turned to -90 degrees
- moved R11 120.8 mm to (173.4, 132.9), turned to 180 degrees
- moved L3 118.7 mm to (46.8, 83.6), turned to -90 degrees
- moved SW1 118.7 mm to (167.9, 138.1)
- moved U7 118.2 mm to (46.6, 78.4), turned to -90 degrees
- moved R41 116.6 mm to (151.0, 125.5), turned to 180 degrees
- moved R10 116.5 mm to (161.5, 134.6)
- moved R42 114.9 mm to (150.9, 121.8), turned to 180 degrees
- moved C22 114.1 mm to (151.8, 138.2)
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Connections:
- J1 pad 170: SPARE_P170 -> HPOUTL
- J1 pad 171: SPARE_P171 -> MICLP
- J1 pad 172: SPARE_P172 -> GND
- J1 pad 58: HPOUTL -> GND
- J1 pad 64: MIPI0_D0N -> MIPI0_CLKP
- J1 pad 65: MIPI0_D0P -> MIPI0_CLKN
- J1 pad 67: MIPI0_D1N -> MIPI0_D1P
- J1 pad 68: MIPI0_D1P -> MIPI0_D1N
- J1 pad 70: MIPI0_CLKN -> MIPI0_D0P
- J1 pad 71: MIPI0_CLKP -> MIPI0_D0N
- J1 pad 77: MIPI1_D0N -> MIPI1_CLKP
- J1 pad 78: MIPI1_D0P -> MIPI1_CLKN
- J1 pad 80: MIPI1_D1N -> MIPI1_D1P
- J1 pad 81: MIPI1_D1P -> MIPI1_D1N
- J1 pad 83: MIPI1_CLKN -> MIPI1_D0P
- J1 pad 84: MIPI1_CLKP -> MIPI1_D0N
- J31 pad 10: SPARE_P178 -> SPARE_P181
- J31 pad 11: SPARE_P179 -> SPARE_P182
- J31 pad 12: SPARE_P180 -> SPARE_P183
- J31 pad 13: SPARE_P181 -> SPARE_P184
- J31 pad 14: SPARE_P182 -> SPARE_P185
- J31 pad 15: SPARE_P183 -> SPARE_P186
- J31 pad 16: SPARE_P184 -> SPARE_P187
- J31 pad 17: SPARE_P185 -> SPARE_P188
- J31 pad 18: SPARE_P186 -> SPARE_P189
- J31 pad 19: SPARE_P187 -> SPARE_P190
- J31 pad 2: SPARE_P170 -> SPARE_P173
- J31 pad 20: SPARE_P188 -> SPARE_P191
- J31 pad 21: SPARE_P189 -> SPARE_P192
- J31 pad 22: SPARE_P190 -> GND
- J31 pad 3: SPARE_P171 -> SPARE_P174
- J31 pad 4: SPARE_P172 -> SPARE_P175
- J31 pad 5: SPARE_P173 -> SPARE_P176
- J31 pad 6: SPARE_P174 -> SPARE_P177
- J31 pad 7: SPARE_P175 -> SPARE_P178
- J31 pad 8: SPARE_P176 -> SPARE_P179
- J31 pad 9: SPARE_P177 -> SPARE_P180
- J6 pad R1: unconnected-(J6-PadR1) -> HPOUTL
- J6 pad R2: unconnected-(J6-PadR2) -> GND
- J6 pad S: unconnected-(J6-PadS) -> MICLP
- J7 pad 1: GND -> +3V3
- J7 pad 10: MIPI0_D1N -> MIPI0_D1P
- J7 pad 11: MIPI0_D1P -> MIPI0_D1N
- J7 pad 13: MIPI0_CLKN -> MIPI0_D0P
- J7 pad 14: MIPI0_CLKP -> MIPI0_D0N
- J7 pad 2: MIPI0_GPIO -> MIPI0_SCCB_SDA
- J7 pad 3: MIPI0_SCCB_SDA -> MIPI0_SCCB_SCL
- J7 pad 4: MIPI0_SCCB_SCL -> +3V3
- J7 pad 5: +3V3 -> MIPI0_SENSOR_EN
- J7 pad 7: MIPI0_D0N -> MIPI0_CLKP
- J7 pad 8: MIPI0_D0P -> MIPI0_CLKN
- J8 pad 1: GND -> +3V3
- J8 pad 10: MIPI1_D1N -> MIPI1_D1P
- J8 pad 11: MIPI1_D1P -> MIPI1_D1N
- J8 pad 13: MIPI1_CLKN -> MIPI1_D0P
- J8 pad 14: MIPI1_CLKP -> MIPI1_D0N
- J8 pad 2: MIPI1_GPIO -> MIPI1_SCCB_SDA
- J8 pad 3: MIPI1_SCCB_SDA -> MIPI1_SCCB_SCL
- J8 pad 4: MIPI1_SCCB_SCL -> +3V3
- J8 pad 5: +3V3 -> MIPI1_SENSOR_EN
- J8 pad 7: MIPI1_D0N -> MIPI1_CLKP
- J8 pad 8: MIPI1_D0P -> MIPI1_CLKN
- SW2 pad 1: EN_SW_BMC -> EN_SW_ALT
- SW2 pad 4: EN_SW_ALT -> EN_SW_BMC
Routing:
- added copper zone on B.Cu, net GND
- added copper zone on F.Cu, net GND
Other:
- board size 280 x 240 mm -> 257 x 117.5 mm
- board text added: "GMAC0"
- board text added: "GMAC1"
- board text added: "GPIO"
- board text added: "PWM"
- board text added: "SAR-ADC"
- board text added: "SMB"
- board text added: "SPARE1"
- board text added: "SPARE2"
- board text added: "SPARE3"
- board text added: "SPARE4"
- board text added: "SPARE5"
- board text added: "SSI0"
- board text added: "SSI1"
- board text added: "UART0"
- board text added: "UART1"
- board text added: "UART2"
- board text added: "UART3"
