File: hw/sheets/power.kicad_sch (KiCad schematic)
At the start: 70 parts, among them U1 AP62600SJ-7, U14 TPS22990DMLR, U2 AP62300WU-7, U3 MCP4661-104E_ST, U4 TPS22990DMLR, U5 AZ1117CH-3.3TRG1, U6 AZ1117CH-1.8TRG1, U7 AP62300WU-7

Commit message: Fix D1/D2 and U13 footprint references (didn't exist in any library)
Found while auditing every footprint reference in CONNECTIONS.txt against
the actual installed libraries (fp-lib-table + on-disk .kicad_mod files),
prompted by the earlier PCB pass's substituted-footprint workaround note:

- D1/D2 (PMEG2010ER): hardcoded Diode_SMD:D_SOD-123W, which doesn't exist
  anywhere, and Diode_SMD wasn't even registered in fp-lib-table. Fixed to
  Diode_SMD:Nexperia_CFP3_SOD-123W (the real footprint for this Nexperia
  part's actual package) and registered the library.
- U13 (W25Q32JVSS): hardcoded Package_SO:SOIC-8_5.23x5.23mm_P1.27mm --
  close but not the real footprint name, Package_SO:SOIC-8_5.3x5.3mm_P1.27mm.

Verified: netlist diff shows only these 3 footprint string changes,
nothing else moved (component count, all pin-net assignments unchanged).
ERC footprint_link_issues: 3 -> 0, no other category changed. PCB rebuild:
still just the 1 expected J6 case, DRC unchanged at 20 pre-existing
fine-pitch clearance violations. Schematic quadrant layout still at 0mm
drift.
Parts:
- D1, D2: footprint Diode_SMD:D_SOD-123W -> Diode_SMD:Nexperia_CFP3_SOD-123W
Changed lines of the file:
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@@
 		(property "Reference" "D1" (at 137.16 8.889999999999999 0) (effects (font (size 1.27 1.27))))
 		(property "Value" "PMEG2010ER" (at 137.16 16.509999999999998 0) (effects (font (size 1.27 1.27))))
-		(property "Footprint" "Diode_SMD:D_SOD-123W" (at 137.16 12.7 0) (effects (font (size 1.27 1.27)) hide))
+		(property "Footprint" "Diode_SMD:Nexperia_CFP3_SOD-123W" (at 137.16 12.7 0) (effects (font (size 1.27 1.27)) hide))
 	)
 	(symbol (lib_id "Device:D_Schottky") (at 137.16 27.94 0) (unit 1)
 		(property "Reference" "D2" (at 137.16 24.130000000000003 0) (effects (font (size 1.27 1.27))))
 		(property "Value" "PMEG2010ER" (at 137.16 31.75 0) (effects (font (size 1.27 1.27))))
-		(property "Footprint" "Diode_SMD:D_SOD-123W" (at 137.16 27.94 0) (effects (font (size 1.27 1.27)) hide))
+		(property "Footprint" "Diode_SMD:Nexperia_CFP3_SOD-123W" (at 137.16 27.94 0) (effects (font (size 1.27 1.27)) hide))
 	)
 	(symbol (lib_id "Regulator_Linear:L7805") (at 190.5 20.32 0) (unit 1)

Commit message: Confirm C13/C23 at 1nF, drop the _TBD marker
C13/C23 set the slew-rate/inrush-limiting CT capacitor on U4/U14
(TPS22990DMLR load switches, SS9). Verified 1nF against TI's own
TPS22990 datasheet, which uses this same 1000pF value as its reference
design default for this exact pin -- the placeholder wasn't wrong, just
unconfirmed against the datasheet until now.

Verified: netlist diff shows only these 2 value string changes, zero
pin-net changes. ERC unchanged at 429 violations. Schematic layout still
at 0mm drift.
Parts:
- C13, C23: value 1nF_TBD -> 1nF
Changed lines of the file:
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@@
 	(symbol (lib_id "Device:C") (at 167.64 121.92 0) (unit 1)
 		(property "Reference" "C13" (at 172.72 120.65 0) (effects (font (size 1.27 1.27))))
-		(property "Value" "1nF_TBD" (at 172.72 123.19 0) (effects (font (size 1.27 1.27))))
+		(property "Value" "1nF" (at 172.72 123.19 0) (effects (font (size 1.27 1.27))))
 		(property "Footprint" "Capacitor_SMD:C_0402_1005Metric" (at 167.64 121.92 0) (effects (font (size 1.27 1.27)) hide))
 	)
@@
 	(symbol (lib_id "Device:C") (at 243.84 121.92 0) (unit 1)
 		(property "Reference" "C23" (at 248.92000000000002 120.65 0) (effects (font (size 1.27 1.27))))
-		(property "Value" "1nF_TBD" (at 248.92000000000002 123.19 0) (effects (font (size 1.27 1.27))))
+		(property "Value" "1nF" (at 248.92000000000002 123.19 0) (effects (font (size 1.27 1.27))))
 		(property "Footprint" "Capacitor_SMD:C_0402_1005Metric" (at 243.84 121.92 0) (effects (font (size 1.27 1.27)) hide))
 	)
