File: hw/sheets/headers.kicad_sch (KiCad schematic)
At the start: 16 parts, among them J20 HDR_J20, J21 HDR_J21, J22 HDR_J22, J23 HDR_J23, J24 HDR_J24, J25 HDR_J25, J26 HDR_J26, J27 HDR_J27, J28 HDR_J28, J29 HDR_J29, J30 HDR_J30, J31 HDR_J31, J32 HDR_J32, J33 HDR_J33, J34 HDR_J34, J35 HDR_J35

Commit message: Carrier board: audio/FPC pinout fixes matching 3.3, SW2 remap, UART1 breakout, real PCB layout
Schematic fixes (verified pin-for-pin against TeaCup(C)3.3's real netlist,
not assumed):
- J6 audio jack: R1/R2 -> HPOUTL/GND, S -> MICLP, matching 3.3's J10 exactly
  (previous wiring incorrectly tied GND to a schematic pin, G, with no
  matching pad on the real Jack_3.5mm_PJ320D_Horizontal footprint).
- J7/J8 FPC camera connectors: full pin-for-pin remap to match 3.3's real
  J13 pinout -- the previous "standard RPi/Arducam" pinout had power/ground
  swapped, clock/data lanes in the wrong order, and reversed differential
  polarity throughout. Added JP11/JP12 sensor-enable select jumpers
  (GPIO vs hardwired +3V3), replicating 3.3's J15.
- J1 MIPI0/MIPI1 pin order on the connector reordered (CLK/D1/D0, P-before-N)
  to match J7/J8's now-fixed order, so routing between them doesn't need to
  cross over itself.
- HPOUTL relocated from J1 pin 58 (isolated, far from any other audio net)
  down to sit beside MICLP at pins 170-172, geography-first per
  UNIVERSAL.md SS8.
- SW2 (manual power-override switch) throw1/throw4 swapped: throw1 now
  forces ALT, throw4 now forces BMC.
- New J36 header breaks out UART1 (the BMC-ESP32<->J1 console link) for
  external monitoring, same as UART0/2/3 already had.

All verified via isolated before/after ERC diffs -- each change nets to
either 0 or a fully-explained delta against the 429-violation baseline,
never an unexplained regression.

PCB: teacup-carrier.kicad_pcb replaced with the manually-laid-out board
(previously developed as a separate merge-test attempt): real component
placement grouped by circuit block, board outline resized twice to
snugly enclose the layout, GND copper pour on both F.Cu and B.Cu, and
mounting holes repositioned to match. The old rough auto-placed board is
gone.
Parts:
- removed J31: HDR_J31, Connector_PinHeader_2.54mm:PinHeader_2x12_P2.54mm_Vertical, symbol Connector_Generic:Conn_02x12_Odd_Even
- added J31: HDR_J31, Connector_PinHeader_2.54mm:PinHeader_2x11_P2.54mm_Vertical, symbol Connector_Generic:Conn_02x11_Odd_Even
- added J36: HDR_J36, Connector_PinHeader_2.54mm:PinHeader_1x03_P2.54mm_Vertical, symbol Connector_Generic:Conn_01x03
Connections:
- net GND: now also J31.1 (Pin_1), J31.22 (Pin_22), J36.1 (Pin_1)
- net SPARE_P173: now also J31.2 (Pin_2)
- net SPARE_P174: now also J31.3 (Pin_3)
- net SPARE_P175: now also J31.4 (Pin_4)
- net SPARE_P176: now also J31.5 (Pin_5)
- net SPARE_P177: now also J31.6 (Pin_6)
- net SPARE_P178: now also J31.7 (Pin_7)
- net SPARE_P179: now also J31.8 (Pin_8)
- net SPARE_P180: now also J31.9 (Pin_9)
- net SPARE_P181: now also J31.10 (Pin_10)
- net SPARE_P182: now also J31.11 (Pin_11)
- net SPARE_P183: now also J31.12 (Pin_12)
- net SPARE_P184: now also J31.13 (Pin_13)
- net SPARE_P185: now also J31.14 (Pin_14)
- net SPARE_P186: now also J31.15 (Pin_15)
- net SPARE_P187: now also J31.16 (Pin_16)
- net SPARE_P188: now also J31.17 (Pin_17)
- net SPARE_P189: now also J31.18 (Pin_18)
- net SPARE_P190: now also J31.19 (Pin_19)
- net SPARE_P191: now also J31.20 (Pin_20)
- net SPARE_P192: now also J31.21 (Pin_21)
- new net UART1_RX: J36.2 (Pin_2)
- new net UART1_TX: J36.3 (Pin_3)
Other:
- note added: "J1 SPARE (P173-192)"
- note added: "UART1 (BMC console)"
- note removed: "J1 SPARE (P170-192)"
