File: hw/.history/teacup-carrier.kicad_pcb (KiCad board)
At the start: 4 copper layers, 257 x 117.5 mm, 138 parts, among them J1 AH58893-T9B10-3F, J2 TYPE-C-31-M-12, J20 HDR_J20, J21 HDR_J21, J22 HDR_J22, J23 HDR_J23, J24 HDR_J24, J25 HDR_J25, J26 HDR_J26, J27 HDR_J27, J28 HDR_J28, J29 HDR_J29, J3 TE_292303-7, J30 HDR_J30, J31 HDR_J31, J32 HDR_J32, J33 HDR_J33, J34 HDR_J34, J35 HDR_J35, J36 HDR_J36, J37 HDR_J37, J38 AMP_MIC_TAP, J4 Hirose_DM3D-SF, J5 Wuerth_694106301002, J6 AudioJack4_Ground, J7 SFW15R-2STE1LF, J8 SFW15R-2STE1LF, J9 TYPE-C-31-M-12, Q1 AO3401A, Q2 AO3401A, SW1 SSSS711403, SW2 SSSS711403, U1 AP62600SJ-7, U10 TS5A3166, U11 DIP-8 Socket, U12 TPS2053BDR, U13 W25Q32JVSS, U14 TPS22990DMLR, U15 TCA9555PWR, U2 AP62300WU-7, U3 MCP4661-104E_ST, U4 TPS22990DMLR, U5 AZ1117CH-3.3TRG1, U6 AZ1117CH-1.8TRG1, U7 AP62300WU-7, U8 ESP32-S3-WROOM-1-N16R2, U9 TS5A3166

Commit message: Remove two degenerate zero-size GND vias near R26
Both had size 0 / drill ~0 (no real copper or hole at all) and were
flagged by DRC as annular_width, drill_out_of_range, via_diameter, and
hole_to_hole violations. Confirmed via DRC diff: only these vias'
associated violations resolved, nothing else on the board changed.
Parts:
- removed C20: 10uF, Capacitor_SMD:C_0805_2012Metric
- moved R8 99.9 mm to (138.8, 94.5)
- moved R42 96.2 mm to (136.3, 91.0)
- moved R41 96.2 mm to (135.7, 93.2), turned to 90 degrees
- moved C21 89.3 mm to (132.5, 111.1)
- moved C22 89.2 mm to (132.0, 114.7)
- moved U11 73.2 mm to (147.9, 131.0), turned to 0 degrees
- moved C15 70.5 mm to (127.9, 110.4), turned to -90 degrees
- moved C14 70.1 mm to (128.2, 114.6), turned to 90 degrees
- moved U12 58.3 mm to (98.5, 103.8)
- moved U15 58.3 mm to (98.4, 91.5)
- moved U13 56.9 mm to (151.8, 121.1), turned to 0 degrees
- moved U5 56.9 mm to (121.3, 112.2), turned to 180 degrees
- moved R9 56.1 mm to (111.4, 81.0), turned to -90 degrees
- moved C24 53.7 mm to (155.1, 116.2), turned to 180 degrees
- moved C16 47.8 mm to (97.3, 112.7), turned to 0 degrees
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Routing:
- net +5V_SW: track 2.83 -> 194.5 mm, vias 0 -> 11
- net USBA_HOST_DM: track 0.00 -> 117.0 mm, vias 0 -> 4
- net USBA_HOST_DP: track 0.00 -> 112.6 mm, vias 0 -> 4
- net SFC_IO2: track 21.5 -> 123.3 mm, vias 0 -> 1
- net SW_SENSE_4: track 0.00 -> 95.5 mm, vias 0 -> 2
- net SW_SENSE_1: track 0.00 -> 91.7 mm, vias 0 -> 2
- net VDDR: track 49.7 -> 136.7 mm, vias 0 -> 2
- net DCJACK_PRESENT: track 0.00 -> 84.9 mm, vias 0 -> 3
- net I2C_PWR_SCL: track 0.00 -> 84.5 mm, vias 0 -> 4
- net I2C_PWR_SDA: track 0.00 -> 83.9 mm, vias 0 -> 4
- net SFC_IO0: track 23.0 -> 98.5 mm, vias 0 -> 2
- net SFC_CLK: track 22.5 -> 96.8 mm, vias 0 -> 2
- net SFC_IO1: track 22.1 -> 93.1 mm, vias 0 -> 2
- net SFC_IO3: track 23.7 -> 94.4 mm, vias 0 -> 2
- net PG_SW5V_ALT: track 0.00 -> 68.4 mm, vias 0 -> 4
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
Commit message: Add GND plane on In2.Cu, fix U4/U14 footprint mismatch, resolve silkscreen overlaps, restore 0.15mm clearance rule
- Added a GND pour on In2.Cu (previously empty) mirroring the F.Cu/B.Cu
  GND zones. Since every via on this board is a full F.Cu-B.Cu through-via
  and several ground-anchoring parts use through-hole pads, this ties
  together fill regions that were fragmented across the outer layers by
  the dense single-layer routing. One remaining isolated region (near
  C15/U5/C14, anchored only by SMD pads with nothing reaching it) got a
  dedicated stitching via. Resolves the "zone vs itself" unconnected-item
  DRC error.
- Refreshed U4/U14 (WSON-10_L3.0-W2.0-P0.50-BL-EP_TI_DML) from the current
  library master -- equivalent to "Update Footprint from Library" --
  resolving lib_footprint_mismatch. Position, orientation, schematic-symbol
  path link, and every pad's net assignment verified identical before and
  after. Also upgraded the library footprint file itself from legacy
  KiCad-6 module syntax to the current format (same content, side effect
  of loading it via the scripting API).
- Resolved the large majority of silk_overlap/silk_over_copper DRC
  warnings by nudging reference-designator text away from whatever it
  was overlapping (another footprint's silkscreen, a pad, or another
  reference field), verified via DRC diff at each step.
- Set the board's minimum clearance rule back to 0.15mm (was raised to
  0.2mm at some point, which retroactively flagged ~90 header-breakout
  traces that were routed under the original 0.15mm rule).

silk_edge_clearance violations (component body silkscreen overhanging
the board edge -- not text, out of scope here) and the two remaining
U4/U14 pad10/11 clearance violations (inherent to that package's real
lead pitch, not fixable by rerouting) are left as-is.
Parts:
- U14, U4: footprint teacup-carrier:WSON-10_L3.0-W2.0-P0.50-BL-EP_TI_DML -> WSON-10_L3.0-W2.0-P0.50-BL-EP_TI_DML
- moved R24 0.68 mm to (117.7, 126.7)
- moved H2 0.36 mm to (271.7, 27.7)
- moved H4 0.36 mm to (271.7, 138.5)
- moved H1 0.36 mm to (21.4, 27.7)
- moved H3 0.36 mm to (21.4, 138.5)
- moved R42 0.09 mm to (136.2, 91.0)
Routing:
- net GND: track 13.8 -> 91.5 mm, vias 17 -> 46
- net SPARE_P220: track 32.7 -> 31.1 mm
- net SPARE_P244: track 39.5 -> 38.3 mm
- net SPARE_P266: track 59.4 -> 58.4 mm
- net SSI0_GPC: track 87.3 -> 88.3 mm
- net SPARE_P248: track 42.2 -> 41.4 mm
- net SPARE_P250: track 43.3 -> 42.5 mm
- net SPARE_P246: track 41.5 -> 40.7 mm
- net SPARE_P210: track 27.6 -> 26.8 mm
- net SPARE_P282: track 62.1 -> 61.5 mm
- added copper zone on In2.Cu, net GND
